Commit message: urdf bottom scratch start

File: src/test_urdf/urdf/test_urdf.urdf.xacro (robot description, xacro)
@@ -3,6 +3,7 @@
      Commit Version: 1.5.1-0-g916b5db  Build Version: 1.5.7152.31018
      For more information, please see http://wiki.ros.org/sw_urdf_exporter -->
-<robot
-  name="test_urdf">
+<robot name="test_urdf" xmlns:xacro="http://www.ros.org/wiki/xacro">
+  <!--xacro variables-->
+  <xacro:property name="PI" value="3.1415926535897931" />
   <!--For base Foot Print-->
   <link name="world"/>
@@ -504,83 +505,3 @@
     <selfCollide>true</selfCollide>
   </gazebo>
-  <transmission name="tran1">
-    <type>transmission_interface/SimpleTransmission</type>
-    <joint name="joint1">
-      <hardwareInterface>hardware_interface/EffortJointInterface</hardwareInterface>
-    </joint>
-    <actuator name="motor1">
-      <hardwareInterface>hardware_interface/EffortJointInterface</hardwareInterface>
-      <mechanicalReduction>1</mechanicalReduction>
-    </actuator>
-  </transmission>
-  <transmission name="tran2">
-    <type>transmission_interface/SimpleTransmission</type>
-    <joint name="joint2">
-      <hardwareInterface>hardware_interface/EffortJointInterface</hardwareInterface>
-    </joint>
-    <actuator name="motor2">
-      <hardwareInterface>hardware_interface/EffortJointInterface</hardwareInterface>
-      <mechanicalReduction>1</mechanicalReduction>
-    </actuator>
-  </transmission>
-  <transmission name="tran3">
-    <type>transmission_interface/SimpleTransmission</type>
-    <joint name="joint3">
-      <hardwareInterface>hardware_interface/EffortJointInterface</hardwareInterface>
-    </joint>
-    <actuator name="motor3">
-      <hardwareInterface>hardware_interface/EffortJointInterface</hardwareInterface>
-      <mechanicalReduction>1</mechanicalReduction>
-    </actuator>
-  </transmission>
-  <transmission name="tran4">
-    <type>transmission_interface/SimpleTransmission</type>
-    <joint name="joint4">
-      <hardwareInterface>hardware_interface/EffortJointInterface</hardwareInterface>
-    </joint>
-    <actuator name="motor4">
-      <hardwareInterface>hardware_interface/EffortJointInterface</hardwareInterface>
-      <mechanicalReduction>1</mechanicalReduction>
-    </actuator>
-  </transmission>
-  <transmission name="tran5">
-    <type>transmission_interface/SimpleTransmission</type>
-    <joint name="joint5">
-      <hardwareInterface>hardware_interface/EffortJointInterface</hardwareInterface>
-    </joint>
-    <actuator name="motor5">
-      <hardwareInterface>hardware_interface/EffortJointInterface</hardwareInterface>
-      <mechanicalReduction>1</mechanicalReduction>
-    </actuator>
-  </transmission>
-  <transmission name="tran6">
-    <type>transmission_interface/SimpleTransmission</type>
-    <joint name="joint6">
-      <hardwareInterface>hardware_interface/EffortJointInterface</hardwareInterface>
-    </joint>
-    <actuator name="motor6">
-      <hardwareInterface>hardware_interface/EffortJointInterface</hardwareInterface>
-      <mechanicalReduction>1</mechanicalReduction>
-    </actuator>
-  </transmission>
-  <transmission name="tran7">
-    <type>transmission_interface/SimpleTransmission</type>
-    <joint name="joint7">
-      <hardwareInterface>hardware_interface/EffortJointInterface</hardwareInterface>
-    </joint>
-    <actuator name="motor7">
-      <hardwareInterface>hardware_interface/EffortJointInterface</hardwareInterface>
-      <mechanicalReduction>1</mechanicalReduction>
-    </actuator>
-  </transmission>
-  <transmission name="tran8">
-    <type>transmission_interface/SimpleTransmission</type>
-    <joint name="joint8">
-      <hardwareInterface>hardware_interface/EffortJointInterface</hardwareInterface>
-    </joint>
-    <actuator name="motor8">
-      <hardwareInterface>hardware_interface/EffortJointInterface</hardwareInterface>
-      <mechanicalReduction>1</mechanicalReduction>
-    </actuator>
-  </transmission>
 </robot>

Commit message: xacro start

File: src/test_urdf/urdf/test_urdf.urdf.xacro (robot description, xacro)
@@ -6,26 +6,64 @@
   <!--xacro variables-->
   <xacro:property name="PI" value="3.1415926535897931" />
+  <xacro:property name="box_width" value="0.050" />
+  <xacro:property name="box_depth" value="0.040" />
+  <xacro:property name="box_height" value="0.080" />
+  <xacro:property name="origin_to_joint_x" value="0" />
+  <xacro:property name="origin_to_joint_y" value="0" />
+  <xacro:property name="origin_to_joint_z" value="-0.014" />
+  <material name="light_grey"><color rgba="0.4 0.4 0.4 1.0" /></material>
+  <!--xacro macro-->
+  <xacro:macro name="node" params="prefix">
+    <link name="${prefix}_link">
+      <visual>
+        <origin xyz="0 0 0" rpy="0 0 0"/>
+        <geometry>
+          <mesh filename="package://test_urdf/meshes/link1.STL" />
+        </geometry>
+        <material name="light_grey" />
+      </visual>
+      <collision>
+        <origin xyz="0 0 0" rpy="0 0 0"/>
+        <geometry>
+          <box size="${box_width} ${box_depth} ${box_height}"/>
+        </geometry>
+      </collision>
+      <inertial>
+        <origin xyz="0 0 0" rpy="0 0 0"/>
+        <mass value="0.060"/>
+        <inertia ixx="4.0E-05" iyy="4.45E-05" izz="2.05E-05"/>
+      </inertial>
+    </link>
+    <!-- <gazebo reference="${prefix}_link">
+      <material>Gazebo/DarkGrey</material>
+      <selfCollide>false</selfCollide>
+      <mu1 value="0.5"/>
+      <mu2 value="0.5"/>
+      <kp value="10000000.0" />
+      <kd value="1" />
+      <fdir1 value="1 0 0"/>
+    </gazebo> -->
+    <joint name="${prefix}_joint" type="continuous">
+      <axis xyz="1 0 0" />
+    </joint>
+    <transmission name="${prefix}_joint_trans">
+      <type>transmission_interface/SimpleTransmission</type>
+      <joint name="${prefix}_joint">
+        <hardwareInterface>hardware_interface/VelocityJointInterface</hardwareInterface>
+      </joint>
+      <actuator name="${prefix}_actuator">
+        <mechanicalReduction>1</mechanicalReduction>
+      </actuator>
+    </transmission>
+  </xacro:macro>
   <!--For base Foot Print-->
-  <link name="world"/>
-  <joint name="floating" type="floating">
-    <parent link="world"/>
-    <child link="base_link"/>
-    <origin xyz="0.0 0.0 0.5" rpy="0 0 0"/>
-  </joint>
-  <link
-    name="base_link">
+  <link name="base_link">
     <inertial>
       <origin
-        xyz="0.0018507 -0.0013143 -0.29442"
+        xyz="0 0 0"
         rpy="0 0 0" />
       <mass
-        value="0.56176" />
-      <inertia
-        ixx="0.016641"
-        ixy="8.8434E-07"
-        ixz="0.00012368"
-        iyy="0.016639"
-        iyz="-0.0001224"
-        izz="9.3717E-05" />
+        value="0.06" />
+      <inertia ixx="4.0E-05" iyy="4.45E-05" izz="2.05E-05"/>
     </inertial>
     <visual>
@@ -37,445 +75,70 @@
           filename="package://test_urdf/meshes/base_link.STL" />
       </geometry>
-      <material
-        name="">
-        <color
-          rgba="0.79216 0.81961 0.93333 1" />
-      </material>
+      <material name="light_grey" />
     </visual>
     <collision>
-      <origin
-        xyz="0 0 0"
-        rpy="0 0 0" />
-      <geometry>
-        <mesh
-          filename="package://test_urdf/meshes/base_link.STL" />
-      </geometry>
+        <origin xyz="0 0 0" rpy="0 0 0"/>
+        <geometry>
+          <box size="${box_width} ${box_depth} ${box_height}"/>
+        </geometry>
     </collision>
   </link>
-  <link
-    name="link1">
-    <inertial>
-      <origin
-        xyz="0.0013143 -0.21542 -0.0018507"
-        rpy="0 0 0" />
-      <mass
-        value="0.56176" />
-      <inertia
-        ixx="0.016639"
-        ixy="0.0001224"
-        ixz="8.8434E-07"
-        iyy="9.3717E-05"
-        iyz="-0.00012368"
-        izz="0.016641" />
-    </inertial>
-    <visual>
-      <origin
-        xyz="0 0 0"
-        rpy="0 0 0" />
-      <geometry>
-        <mesh
-          filename="package://test_urdf/meshes/link1.STL" />
-      </geometry>
-      <material
-        name="">
-        <color
-          rgba="0.79216 0.81961 0.93333 1" />
-      </material>
-    </visual>
-    <collision>
-      <origin
-        xyz="0 0 0"
-        rpy="0 0 0" />
-      <geometry>
-        <mesh
-          filename="package://test_urdf/meshes/link1.STL" />
-      </geometry>
-    </collision>
-  </link>
-  <joint
-    name="joint1"
-    type="continuous">
-    <origin
-      xyz="0 0 -0.079"
-      rpy="1.5708 0 -1.5708" />
-    <parent
-      link="base_link" />
-    <child
-      link="link1" />
-    <axis
-      xyz="0 0 1" />
-  </joint>
-  <link
-    name="link2">
-    <inertial>
-      <origin
-        xyz="-0.00085074 -0.14792 -0.0013143"
-        rpy="0 0 0" />
-      <mass
-        value="0.56176" />
-      <inertia
-        ixx="0.016641"
-        ixy="-0.00012368"
-        ixz="-8.8434E-07"
-        iyy="9.3717E-05"
-        iyz="-0.0001224"
-        izz="0.016639" />
-    </inertial>
-    <visual>
-      <origin
-        xyz="0 0 0"
-        rpy="0 0 0" />
-      <geometry>
-        <mesh
-          filename="package://test_urdf/meshes/link2.STL" />
-      </geometry>
-      <material
-        name="">
-        <color
-          rgba="0.79216 0.81961 0.93333 1" />
-      </material>
-    </visual>
-    <collision>
-      <origin
-        xyz="0 0 0"
-        rpy="0 0 0" />
-      <geometry>
-        <mesh
-          filename="package://test_urdf/meshes/link2.STL" />
-      </geometry>
-    </collision>
-  </link>
-  <joint
-    name="joint2"
-    type="continuous">
-    <origin
-      xyz="0 -0.0675 -0.001"
-      rpy="0 -1.5708 0" />
-    <parent
-      link="link1" />
-    <child
-      link="link2" />
-    <axis
-      xyz="0 0 1" />
-  </joint>
-  <link
-    name="link3">
-    <inertial>
-      <origin
-        xyz="0.00031427 -0.080424 -0.00085074"
-        rpy="0 0 0" />
-      <mass
-        value="0.56176" />
-      <inertia
-        ixx="0.016639"
-        ixy="0.0001224"
-        ixz="8.8434E-07"
-        iyy="9.3717E-05"
-        iyz="-0.00012368"
-        izz="0.016641" />
-    </inertial>
-    <visual>
-      <origin
-        xyz="0 0 0"
-        rpy="0 0 0" />
-      <geometry>
-        <mesh
-          filename="package://test_urdf/meshes/link3.STL" />
-      </geometry>
-      <material
-        name="">
-        <color
-          rgba="0.79216 0.81961 0.93333 1" />
-      </material>
-    </visual>
-    <collision>
-      <origin
-        xyz="0 0 0"
-        rpy="0 0 0" />
-      <geometry>
-        <mesh
-          filename="package://test_urdf/meshes/link3.STL" />
-      </geometry>
-    </collision>
-  </link>
-  <joint
-    name="joint3"
-    type="continuous">
-    <origin
-      xyz="0 -0.0675 -0.001"
-      rpy="0 1.5708 0" />
-    <parent
-      link="link2" />
-    <child
-      link="link3" />
-    <axis
-      xyz="0 0 1" />
-  </joint>
-  <link
-    name="link4">
-    <inertial>
-      <origin
-        xyz="0.00014926 -0.012924 -0.00031427"
-        rpy="0 0 0" />
-      <mass
-        value="0.56176" />
-      <inertia
-        ixx="0.016641"
-        ixy="-0.00012368"
-        ixz="-8.8434E-07"
-        iyy="9.3717E-05"
-        iyz="-0.0001224"
-        izz="0.016639" />
-    </inertial>
-    <visual>
-      <origin
-        xyz="0 0 0"
-        rpy="0 0 0" />
-      <geometry>
-        <mesh
-          filename="package://test_urdf/meshes/link4.STL" />
-      </geometry>
-      <material
-        name="">
-        <color
-          rgba="0.79216 0.81961 0.93333 1" />
-      </material>
-    </visual>
-    <collision>
-      <origin
-        xyz="0 0 0"
-        rpy="0 0 0" />
-      <geometry>
-        <mesh
-          filename="package://test_urdf/meshes/link4.STL" />
-      </geometry>
-    </collision>
-  </link>
-  <joint
-    name="joint4"
-    type="continuous">
-    <origin
-      xyz="0 -0.0675 -0.001"
-      rpy="0 -1.5708 0" />
-    <parent
-      link="link3" />
-    <child
-      link="link4" />
-    <axis
-      xyz="0 0 1" />
-  </joint>
-  <link
-    name="link5">
-    <inertial>
-      <origin
-        xyz="-0.00068573 0.054576 0.00014926"
-        rpy="0 0 0" />
-      <mass
-        value="0.56176" />
-      <inertia
-        ixx="0.016639"
-        ixy="0.0001224"
-        ixz="8.8434E-07"
-        iyy="9.3717E-05"
-        iyz="-0.00012368"
-        izz="0.016641" />
-    </inertial>
-    <visual>
-      <origin
-        xyz="0 0 0"
-        rpy="0 0 0" />
-      <geometry>
-        <mesh
-          filename="package://test_urdf/meshes/link5.STL" />
-      </geometry>
-      <material
-        name="">
-        <color
-          rgba="0.79216 0.81961 0.93333 1" />
-      </material>
-    </visual>
-    <collision>
-      <origin
-        xyz="0 0 0"
-        rpy="0 0 0" />
-      <geometry>
-        <mesh
-          filename="package://test_urdf/meshes/link5.STL" />
-      </geometry>
-    </collision>
-  </link>
-  <joint
-    name="joint5"
-    type="continuous">
-    <origin
-      xyz="0 -0.0675 -0.001"
-      rpy="0 1.5708 0" />
-    <parent
-      link="link4" />
-    <child
-      link="link5" />
-    <axis
-      xyz="0 0 1" />
-  </joint>
-  <link
-    name="link6">
-    <inertial>
-      <origin
-        xyz="0.0011493 0.12208 0.00068573"
-        rpy="0 0 0" />
-      <mass
-        value="0.56176" />
-      <inertia
-        ixx="0.016641"
-        ixy="-0.00012368"
-        ixz="-8.8434E-07"
-        iyy="9.3717E-05"
-        iyz="-0.0001224"
-        izz="0.016639" />
-    </inertial>
-    <visual>
-      <origin
-        xyz="0 0 0"
-        rpy="0 0 0" />
-      <geometry>
-        <mesh
-          filename="package://test_urdf/meshes/link6.STL" />
-      </geometry>
-      <material
-        name="">
-        <color
-          rgba="0.79216 0.81961 0.93333 1" />
-      </material>
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