Commit message: 삽질

File: src/urdfs/test_urdf/urdf/test_urdf.urdf.xacro (robot description, xacro)
@@ -46,4 +46,5 @@
     <joint name="${prefix}_joint" type="continuous">
       <axis xyz="1 0 0" />
+      <xacro:insert_block name="joint_pose" />
     </joint>
     <transmission name="${prefix}_joint_trans">
@@ -85,4 +86,5 @@
   </link>
   <xacro:node prefix="1">
+    <origin xyz="${origin_to_joint_x} ${origin_to_joint_y} ${-origin_to_joint_z}" rpy="0 0 ${PI/4}" />
     <joint>
       <origin xyz="${origin_to_joint_x} ${origin_to_joint_y} ${origin_to_joint_z}" rpy="0 0 0" />
@@ -92,4 +94,5 @@
   </xacro:node>
   <xacro:node prefix="2">
+    <origin xyz="${origin_to_joint_x} ${origin_to_joint_y} ${-origin_to_joint_z}" rpy="0 0 ${-PI/4}" />
     <joint>
       <origin xyz="${origin_to_joint_x} ${origin_to_joint_y} ${origin_to_joint_z}" rpy="0 0 0" />
@@ -99,4 +102,5 @@
   </xacro:node>
   <xacro:node prefix="3">
+    <origin xyz="${origin_to_joint_x} ${origin_to_joint_y} ${-origin_to_joint_z}" rpy="0 0 ${PI/4}" />
     <joint>
       <origin xyz="${origin_to_joint_x} ${origin_to_joint_y} ${origin_to_joint_z}" rpy="0 0 0" />
@@ -106,4 +110,5 @@
   </xacro:node>
   <xacro:node prefix="4">
+    <origin xyz="${origin_to_joint_x} ${origin_to_joint_y} ${-origin_to_joint_z}" rpy="0 0 ${-PI/4}" />
     <joint>
       <origin xyz="${origin_to_joint_x} ${origin_to_joint_y} ${origin_to_joint_z}" rpy="0 0 0" />
@@ -113,4 +118,5 @@
   </xacro:node>
   <xacro:node prefix="5">
+    <origin xyz="${origin_to_joint_x} ${origin_to_joint_y} ${-origin_to_joint_z}" rpy="0 0 ${PI/4}" />
     <joint>
       <origin xyz="${origin_to_joint_x} ${origin_to_joint_y} ${origin_to_joint_z}" rpy="0 0 0" />
@@ -120,4 +126,5 @@
   </xacro:node>
   <xacro:node prefix="6">
+    <origin xyz="${origin_to_joint_x} ${origin_to_joint_y} ${-origin_to_joint_z}" rpy="0 0 ${-PI/4}" />
     <joint>
       <origin xyz="${origin_to_joint_x} ${origin_to_joint_y} ${origin_to_joint_z}" rpy="0 0 0" />
@@ -127,4 +134,5 @@
   </xacro:node>
   <xacro:node prefix="7">
+    <origin xyz="${origin_to_joint_x} ${origin_to_joint_y} ${-origin_to_joint_z}" rpy="0 0 ${PI/4}" />
     <joint>
       <origin xyz="${origin_to_joint_x} ${origin_to_joint_y} ${origin_to_joint_z}" rpy="0 0 0" />
@@ -134,4 +142,5 @@
   </xacro:node>
   <xacro:node prefix="8">
+    <origin xyz="${origin_to_joint_x} ${origin_to_joint_y} ${-origin_to_joint_z}" rpy="0 0 ${-PI/4}" />
     <joint>
       <origin xyz="${origin_to_joint_x} ${origin_to_joint_y} ${origin_to_joint_z}" rpy="0 0 0" />
